File: Hardware/Kicad/base_station_rev1.2_16MAY/base_station.kicad_pcb (KiCad board)
At the start: 2 copper layers, 101 x 57.7 mm, 86 parts, among them CON1 USB-MICRO-B, CON2 AVR-ISP-6, J1 RJ45-CON, P1 CONN_1, P2 CONN_1, P3 CONN_1, P4 CONN_1, Q1 MOS_N, SW1 SW_PUSH, U1 AP7333-33SAG-7, U2 ATMEGA32U4, U3 W5100, U4 RX2004A_BIW, U5 NRF24L01, U6 24AA02E48T-I/OT, X1 8MHz, X2 25MHz

Commit message: Modified HW - BS gerbers
Parts:
- added G***: LOGO, BasestationFP:LOGO, F.Cu at (160.2, 116.5)
- added REF**: Symbol_OSHW-Logo_SilkScreen, Symbols:Symbol_OSHW-Logo_SilkScreen, F.Cu at (169.0, 115.5)
- C1, C10, C11, C12, C13, C14, C15, C16, C17, C18, C2, C21, C22, C23, C24, C25, C26, C27, C28, C29, C3, C30, C31, C32, C33, C34, C35, C36, C37, C38, C39, C4, C40, C41, C42, C5, C6, C7, C8, C9: footprint SM0603_Capa -> BasestationFP:SM0603_Capa
- CON1: footprint con_microusb_10103594 -> BasestationFP:con_microusb_10103594
- CON2: footprint pin_array_3x2 -> BasestationFP:pin_array_3x2
- FB1, FB2, FB3: footprint SM0603 -> BasestationFP:SM0603
- J1: footprint CON_RJ45_TRANSFO -> BasestationFP:CON_RJ45_TRANSFO
- P1: footprint HOLE_FIX_HAMMOND -> BasestationFP:HOLE_FIX_HAMMOND
- Q1: footprint SOT23GDS -> BasestationFP:SOT23GDS
- R1, R10, R11, R12, R13, R14, R15, R16, R17, R18, R19, R2, R20, R3, R4, R5, R6, R7, R8, R9: footprint SM0603_Resistor -> BasestationFP:SM0603_Resistor
- R21, R22: footprint SM0603 -> BasestationFP:SM0603_Resistor
- SW1: footprint SWITCH_FSM16JH -> BasestationFP:SWITCH_FSM16JH
- U1: footprint SOT23 -> BasestationFP:SOT23
- U2: footprint TQFP44 -> BasestationFP:TQFP44
- U3: footprint LQFP80 -> BasestationFP:LQFP80
- U4: footprint LCD_RX200A-BIW -> BasestationFP:LCD_RX200A-BIW
- U5: footprint NRF24L01 -> BasestationFP:NRF24L01
- X1, X2: footprint HC49US -> BasestationFP:HC49US
- moved R5 0.83 mm to (130.2, 103.8)
- turned Q1 to 90 degrees
- turned U1 to 90 degrees
- turned U6 to 270 degrees
Routing:
- net /SPI_nSS: track 53.3 -> 54.2 mm
Other:
- board text added: "HarvestGeek Base Station V1.2"
- board text removed: "Harvestgeek Base Station M. Stephan"
