File: Hardware/Kicad/sensor_station_rev1.2_22MAY/sensor_station.kicad_pcb (KiCad board)
At the start: 2 copper layers, 93.9 x 43.9 mm, 56 parts, among them CON1 USB-MICRO-B, CON2 AVR-ISP-6, K1 CONN_3, P1 CONN_1, P5 CONN_2, SW1 SW_PUSH, U1 AP7333-33SAG-7, U2 ATMEGA32U4, U3 REFERENCE, U4 TSL2581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

Commit message: 23/06/2015 RG
Parts:
- added C18: 100nF, Sensor:SM0603_Capa, F.Cu at (202.1, 159.1)
- added C19: 1uF, Sensor:SM0603_Capa, F.Cu at (202.1, 157.3)
- added C20: 1uF, Sensor:SM0603_Capa, F.Cu at (203.0, 164.8)
- added R14: 10k, Sensor:SM0603_Resistor, F.Cu at (239.0, 186.6)
- added R15: 10k, Sensor:SM0603_Resistor, F.Cu at (238.9, 183.0)
- added U7: AP22802AW5-7, Sensor:AP22802AW5-7, F.Cu at (201.3, 162.0)
- moved C17 14.9 mm to (271.4, 169.9)
Connections:
- CON1 pad 10: GND -> (no net)
- CON1 pad 11: GND -> (no net)
- CON1 pad 4: (no net) -> Net-(CON1-Pad4)
- K1 pad 1: +3.3V -> /SOIL_5V
- U2 pad 1: (no net) -> Net-(U2-Pad1)
- U2 pad 12: (no net) -> Net-(U2-Pad12)
- U2 pad 26: /F_HUMIDITY -> Net-(U2-Pad26)
- U2 pad 27: (no net) -> Net-(U2-Pad27)
- U2 pad 36: (no net) -> Net-(U2-Pad36)
- U2 pad 37: (no net) -> Net-(U2-Pad37)
- U2 pad 38: (no net) -> Net-(U2-Pad38)
- U2 pad 39: (no net) -> Net-(U2-Pad39)
- U2 pad 40: (no net) -> /F_HUMIDITY
- U2 pad 41: (no net) -> /HUM_POWER
- U2 pad 8: (no net) -> /SPI_nSS
- U3 pad 3: (no net) -> Net-(U3-Pad3)
Routing:
- net /SOIL_5V: track 0.00 -> 138.9 mm, vias 0 -> 2
- net /F_HUMIDITY: track 63.4 -> 88.9 mm, vias 0 -> 2
- net /HUM_POWER: track 0.00 -> 25.3 mm, vias 0 -> 2
- net GND: track 62.4 -> 80.4 mm, vias 21 -> 22
- net +5V: track 17.1 -> 26.2 mm
- net +3.3V: track 109.2 -> 104.1 mm
- net Net-(U2-Pad26): track 0.00 -> 0.68 mm
Other:
- board text added: "HarvestGeek Sensor Station Rev 1.3"
- board text added: "RG - 03 July 2014 - Changed outline to fit Polycase SL-30F enclosure - Moved RF module to fit on new outline and ammended keep out areas - Moved switch SW from right to left hand position for continuity with base station - Moved connectors P5, K4 and CON1 to edge of board - Re-routed nets as necessary RG - 01 Aug 2014 - Moved LED D1, R11 and R13 - Re-routed USB traces RG - 22/05/2015 - Modified S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"
- board text removed: "HarvestGeek Sensor Station Rev 1.2"
- board text removed: "Rowan Gifford - 03 July 2014 - Changed outline to fit Polycase SL-30F enclosure - Moved RF module to fit on new outline and ammended keep out areas - Moved switch SW from right to left hand position for continuity with base station - Moved connectors P5, K4 and CON1 to edge of board - Re-routed nets as necessary Rowan Gifford - 01 Aug 2014 - Moved LED D1, R11 and R13 - Re-routed USB traces Rowan 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"
