File: Hardware/Kicad/sensor_station_rev1.2_22MAY/sensor_station.sch (KiCad schematic (older format))
At the start: 51 parts, among them CON1 USB-MICRO-B, CON2 AVR-ISP-6, K1 CONN_3, P1 CONN_1, P2 CONN_1, P3 CONN_1, P4 CONN_1, P5 CONN_2, SW1 SW_PUSH, U1 AP7333-33SAG-7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

Commit message: 23/06/2015 RG
Parts:
- added C18: 100nF, Sensor:SM0603_Capa, symbol C
- added C19, C20: 1uF, Sensor:SM0603_Capa, symbol C
- added R14, R15: 10k, Sensor:SM0603_Resistor, symbol R
- added U7: AP22802AW5-7, Sensor:AP22802AW5-7, symbol AP22802AW5-7
- C1, C10, C11, C12, C13, C14, C15, C16, C17, C2, C3, C33, C36, C39, C4, C5, C6, C7, C8, C9: footprint ~ -> Sensor:SM0603_Capa
- CON1: footprint (none) -> con_microusb_10103594
- CON2: footprint AVR-ISP-6 -> pin_array_3x2
- D1: footprint ~ -> Sensor:LED_BIC_LST
- FB3: footprint ~ -> SM0603
- K1: footprint (none) -> Sensor:CON_3_weidmuller
- P1, P2, P3, P4: footprint (none) -> HOLE_FIX_HAMMOND
- P5: footprint (none) -> CON_2_weidmuller
- R1, R10, R11, R12, R13, R2, R3, R4, R5, R6, R7, R8, R9: footprint ~ -> Sensor:SM0603_Resistor
- SW1: footprint ~ -> SWITCH_FSM16JH
- U1: footprint (none) -> Sensor:SOT23
- U2: footprint ~ -> TQFP44
- U3: footprint (none) -> TO92F
- U4: footprint (none) -> 6-WDFN
- U5: footprint (none) -> NRF24L01
- U6: footprint (none) -> DHT22
- X1: footprint ~ -> HC49US
Connections:
- net labels added: HUM_POWER, SOIL_5V
- wire segments 179 -> 197
Other:
- moved on the sheet: C17, CON1, K1
